File: FC_Internal_v1a/flight_computer_dev_board_rfm98pw.kicad_sch (KiCad schematic)
At the start: 96 parts, among them IC1 RP2040_QFN56, IC2 AZ1117CH-3.3TRG1, J1 Conn_ARM_JTAG_SWD_10, J10 BM04B-SRSS-TB(LF)(SN), J11 BM04B-SRSS-TB(LF)(SN), J12 BM04B-SRSS-TB(LF)(SN), J13 Breakout, J15 Battery, J15 Breakout, J2 FC to EPS Connector, J3 Life Makes Lemonade, J4 104031-0811, J5 BM04B-SRSS-TB(LF)(SN), J6 Conn_Coaxial, J7 Breakout, J8 USB_B_Micro, J9 BM04B-SRSS-TB(LF)(SN), SW1 KMR2, SW2 KMR2, U10 AP3602AKTR-G1, U3 MAX706RESA, U4 RFM98PW, U5 RFM9xBreakout, U6 W25Q128JV, U7 LSM6DSOTR, U8 LSM303AGRTR, U9 MCP25625-E/ML, Y1 12MHZ, Y3 16MHZ 12 pf

Commit message: Major Schematic Refactor
Parts:
- U9: symbol MCP25625-E_ML:MCP25625-E/ML -> MCP25625-E_ML:MCP25625-E/ML
Other:
- note added: "3v3 Linear Regulator"
- note added: "Bus Breakouts"
- note added: "Can Bus"
- note added: "Flash Memory"
- note added: "For USB Power"
- note added: "IMU"
- note added: "SD Card"
- moved on the sheet: C1, C10, C11, C12, C13, C14, C15, C16, C2, C3, C31, C32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
