File: FC_V4b/FC_V4b.kicad_pcb (KiCad board)
At the start: 4 copper layers, 88 x 94.5 mm, 123 parts, among them IC1 RP2040_QFN56, IC2 AZ1117CH-3.3TRG1, IC3 RV-3028-C7_32.768kHz_1ppm_TA_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, J1 Conn_ARM_JTAG_SWD_10, J11 BM04B-SRSS-TB(LF)(SN), J12 BM04B-SRSS-TB(LF)(SN), J13 Breakout, J14 Battery, J15 Breakout, J16 Debug, J2 FC to EPS Connector, J3 Life Makes Lemonade, J4 Molex 503398-1892, J5 BM04B-SRSS-TB(LF)(SN), J6 Conn_Coaxial, J7 Breakout, J8 USB_B_Micro, J9 BM04B-SRSS-TB(LF)(SN), SW1 KMR2, SW2 KMR2, U10 AP3602AKTR-G1, U3 MAX706RESA, U4 RFM98PW, U5 RFM9xBreakout, U6 W25Q128JV, U7 LSM6DSOTR, U8 LSM303AGRTR, U9 MCP25625-E/ML, Y1 12MHZ, Y3 16MHZ 12 pf

Commit message: Finished Layout and Added Artwork
Parts:
- removed J11: BM04B-SRSS-TB(LF)(SN), FC_DEV_BOARD:JST_BM04B-SRSS-TB(LF)(SN)
- C1017, C1018, C1019, C1020, C1021, C1022, C1023, C1024, C1025, C1026, C1027, C1028: moved to F.Cu
- moved C1026 24.6 mm to (180.5, 95.4), turned to 0 degrees
- moved C1027 24.6 mm to (180.5, 99.4), turned to 0 degrees
- moved C1022 21.0 mm to (178.7, 89.9), turned to 45 degrees
- moved C1028 20.0 mm to (178.2, 104.4), turned to -45 degrees
- moved C1018 11.7 mm to (162.4, 94.6), turned to 180 degrees
- moved C1019 11.7 mm to (162.4, 98.6), turned to 180 degrees
- moved C1025 11.1 mm to (173.7, 87.4)
- moved C1023 10.1 mm to (173.2, 106.4)
- moved C1020 8.12 mm to (164.2, 103.9), turned to -135 degrees
- moved C1017 7.14 mm to (164.7, 89.4), turned to 135 degrees
- moved C18 6.65 mm to (170.9, 93.9)
- moved IC3 6.65 mm to (171.4, 97.0)
- moved R14 6.65 mm to (167.9, 96.4)
- moved C17 6.65 mm to (172.4, 95.1)
- moved R5 6.65 mm to (175.7, 95.8)
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Routing:
- net GND: track 246.6 -> 315.5 mm, vias 88 -> 99
- net SCL1: track 83.0 -> 70.7 mm
- net SDA1: track 78.7 -> 67.5 mm
- net RTC_INT: track 71.6 -> 64.5 mm
- net D0: track 68.0 -> 73.3 mm, vias 3 -> 4
- net 3.3V: track 91.5 -> 96.1 mm, vias 36 -> 35
- net RF1_IO0: track 64.9 -> 66.4 mm
- net RF1_IO4: track 61.9 -> 61.3 mm, vias 4 -> 3
- net +5V: track 15.8 -> 16.4 mm
- net VCC_RF1: track 90.7 -> 91.2 mm, vias 5 -> 2
- net V_BACKUP: vias 1 -> 0
- added copper zone on F.Cu, net V_BACKUP
- removed copper zone on B.Cu, net V_BACKUP
Other:
- board text added: "Nebulosity in The Pleiades The Hubble Space Telescope"
- board text added: "PySquared Flight Controller Board V4b By Nicole Maggard & Michael Pham"
- board text removed: "A Total Solar Eclipse"
- board text removed: "DEVELOPERS! DEVELOPERS! DEVELOPERS! DEVELOPERS! DEVELOPERS! DEVELOPERS! DEVELOPERS! DEVELOPERS! DEVELOPERS! DEVELOPERS! DEVELOPERS!"
- board text removed: "PySquared Flight Controller Board V4 By Nicole Maggard & Michael Pham"

Commit message: As Ordered July 17, 2024
Parts:
- added G***: LOGO, LOGO, F.Cu at (200.6, 127.4)
- added REF**: Val**, mainboard:XYZ_cubesat-top, F.Cu at (156.1, 132.4)
- R11: footprint Resistor_SMD:R_0402_1005Metric -> Resistor_SMD:R_0603_1608Metric
- moved R11 0.81 mm to (164.1, 121.7)
Routing:
- net GND: track 315.5 -> 330.2 mm, vias 99 -> 104
- net 3.3V: track 96.1 -> 106.8 mm, vias 35 -> 37
- net SCL1: track 70.7 -> 77.9 mm
- net SDA1: track 67.5 -> 74.0 mm
- net SPI0_CS1: track 77.5 -> 78.1 mm
Other:
- board text added: "BRONCO SPACE Educational Product For Instructional Use Only"
- board text added: "Bridge left for Battery Board V2 Bridge right for camera board"
- board text added: "Do Not Connect 12pos to Battery Board V3"
- board text added: "Hubble Space Telescope Nebulosity in The Pleiades"
- board text added: "Jump to Power via USB Remobe for battery"
- board text added: "Reminder: If RFM9xPW (Large Radio) is used center pads on board must be masked with kapton"
- board text added: "Top Cap Debug"
- board text removed: "Bridge left for battery board Bridge right for camera board"
- board text removed: "Jump to Power via USB"
- board text removed: "Nebulosity in The Pleiades The Hubble Space Telescope"
