File: FC_V5_dev_rev1/sensors.kicad_sch (KiCad schematic)
At the start: 19 parts, among them IC3 RV-3028-C7_32.768kHz_1ppm_TA_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, U12 TCA9548ARGERQ1, U16 MCP9808T-E/MS, U7 LSM6DSOTR, U8 LSM303AGRTR

Commit message: Return of the Shift Register
Parts:
- removed R15: 10K, Resistor_SMD:R_0603_1608Metric, symbol Device:R_US
- removed U12: TCA9548ARGERQ1, TCAQ1:QFN_GERQ1_TEX, symbol TCA9548ARGERQ1:TCA9548ARGERQ1
Connections:
- no-connect marks 18 -> 12
Other:
- note removed: "Sensor Multiplexer"

Commit message: Banished the Shift Register Again for the MCP23017_SS
Other:
- note added: "Real Time Clock"
- moved on the sheet: C31, C32, C33, C34, C35, U7, U8
