File: FC_V5a/watchdog.kicad_sch (KiCad schematic)
At the start: 36 parts, among them U1 TLV1704, U3 AP22652

Commit message: Corrected Load Switch Erratum
The load switch current limit resistors are pulled down now instead of up!
Connections:
- net +3V3: no longer R23.1
- net GND: now also R23.1
Other:
- moved on the sheet: R23
Changed lines of the file:
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@@
 	(wire
 		(pts
-			(xy 118.11 25.4) (xy 118.11 22.86)
+			(xy 111.76 25.4) (xy 111.76 26.67)
 		)
 		(stroke
@@
 	(wire
 		(pts
+			(xy 111.76 31.75) (xy 111.76 34.29)
+		)
+		(stroke
+			(width 0)
+			(type default)
+		)
+	)
+	(wire
+		(pts
 			(xy 110.49 91.44) (xy 110.49 119.38)
 		)
@@
 	(wire
 		(pts
-			(xy 129.54 25.4) (xy 118.11 25.4)
+			(xy 129.54 25.4) (xy 111.76 25.4)
 		)
 		(stroke
@@
 	)
 	(symbol
-		(lib_id "power:+3V3")
-		(at 118.11 17.78 0)
-		(unit 1)
-		(exclude_from_sim no)
-		(in_bom yes)
-		(on_board yes)
-		(dnp no)
-		(property "Reference" "#PWR013"
-			(at 118.11 21.59 0)
-			(effects
-				(font
-					(size 1.27 1.27)
-				)
-				(hide yes)
-			)
-		)
-		(property "Value" "+3V3"
-			(at 114.046 16.51 0)
-			(effects
-				(font
-					(size 1.27 1.27)
-				)
-			)
-		)
-		(property "Footprint" ""
-			(at 118.11 17.78 0)
-			(effects
-				(font
-					(size 1.27 1.27)
-				)
-				(hide yes)
-			)
-		)
-		(property "Datasheet" ""
-			(at 118.11 17.78 0)
-			(effects
-				(font
-					(size 1.27 1.27)
-				)
-				(hide yes)
-			)
-		)
-		(property "Description" "Power symbol creates a global label with name \"+3V3\""
-			(at 118.11 17.78 0)
-			(effects
-				(font
-					(size 1.27 1.27)
-				)
-				(hide yes)
-			)
-		)
-		(pin "1"
-		)
-		(instances
-			(project "FC_V5"
-				(path "/c64c0d72-a9f6-4f3a-891e-1f647558f538/d3e26510-981a-4dd5-9b7d-a587e6324dc6"
-					(reference "#PWR013")
-					(unit 1)
-				)
-			)
-		)
-	)
-	(symbol
 		(lib_id "Device:R_Small_US")
 		(at 190.5 142.24 270)
@@
 	(symbol
 		(lib_id "Device:R_Small_US")
-		(at 118.11 20.32 0)
-		(mirror y)
+		(at 111.76 29.21 0)
+		(mirror x)
 		(unit 1)
 		(exclude_from_sim no)
@@
 		(dnp no)
 		(property "Reference" "R23"
-			(at 112.776 19.05 0)
+			(at 108.966 30.48 0)
 			(effects
 				(font
@@
 		)
 		(property "Value" "47k"
-			(at 112.776 21.844 0)
+			(at 108.966 27.686 0)
 			(effects
 				(font
@@
 		)
 		(property "Footprint" "Resistor_SMD:R_0603_1608Metric"
-			(at 118.11 20.32 0)
+			(at 111.76 29.21 0)
 			(effects
 				(font
@@
 		)
 		(property "Datasheet" "~"
-			(at 118.11 20.32 0)
+			(at 111.76 29.21 0)
 			(effects
 				(font
@@
 		)
 		(property "Description" "47 kOhms ±1% 0.1W, 1/10W Chip Resistor 0603 (1608 Metric) Automotive AEC-Q200 Thick Film"
-			(at 118.11 20.32 0)
+			(at 111.76 29.21 0)
 			(effects
 				(font
@@
 		)
 		(property "DPN" "RMCF0603FT47K0CT-ND"
-			(at 118.11 20.32 0)
+			(at 111.76 29.21 0)
 			(effects
 				(font
@@
 		)
 		(property "DST" "Digi-Key"
-			(at 118.11 20.32 0)
+			(at 111.76 29.21 0)
 			(effects
 				(font
@@
 		)
 		(property "MFR" "Stackpole Electronics Inc"
-			(at 118.11 20.32 0)
+			(at 111.76 29.21 0)
 			(effects
 				(font
@@
 		)
 		(property "MPN" "RMCF0603FT47K0"
-			(at 118.11 20.32 0)
+			(at 111.76 29.21 0)
 			(effects
 				(font
@@
 					(unit 1)
 				)
+			)
+		)
+	)
+	(symbol
+		(lib_name "GND_1")
+		(lib_id "power:GND")
+		(at 111.76 34.29 0)
+		(unit 1)
+		(exclude_from_sim no)
+		(in_bom yes)
+		(on_board yes)
+		(dnp no)
+		(property "Reference" "#PWR0142"
+			(at 111.76 40.64 0)
+			(effects
+				(font
+					(size 1.27 1.27)
+				)
+				(hide yes)
+			)
+		)
+		(property "Value" "GND"
+			(at 107.188 35.814 0)
+			(effects
+				(font
+					(size 1.27 1.27)
+				)
+			)
+		)
+		(property "Footprint" ""
+			(at 111.76 34.29 0)
+			(effects
+				(font
+					(size 1.27 1.27)
+				)
+				(hide yes)
+			)
+		)
+		(property "Datasheet" ""
+			(at 111.76 34.29 0)
+			(effects
+				(font
+					(size 1.27 1.27)
+				)
+				(hide yes)
+			)
+		)
+		(property "Description" "Power symbol creates a global label with name \"GND\" , ground"
+			(at 111.76 34.29 0)
+			(effects
+				(font
+					(size 1.27 1.27)
+				)
+				(hide yes)
+			)
+		)
+		(pin "1"
+		)
+		(instances
+			(project "FC_V5a"
+				(path "/c64c0d72-a9f6-4f3a-891e-1f647558f538/d3e26510-981a-4dd5-9b7d-a587e6324dc6"
+					(reference "#PWR0142")
+					(unit 1)
+				)
