File: FC_V5b/watchdog.kicad_sch (KiCad schematic)
At the start: 36 parts, among them U1 TLV1704, U3 AP22652

Commit message: Changed to AP22653AW6-7 Load Switches for EN High
Parts:
- U3: value AP22652 -> AP22653AW6-7
Changed lines of the file:
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@@
 			)
 		)
-		(property "Value" "AP22652"
+		(property "Value" "AP22653AW6-7"
 			(at 140.97 20.32 0)
 			(effects
