File: FC_V6/load_switches.kicad_sch (KiCad schematic)
At the start: 0 parts

Commit message: Added 3v3 Load Switch Schematic
Parts:
- added C19, C20: 10uF, symbol Device:C
- added U7, U8: TPS22993, Package_DFN_QFN:Texas_S-PWQFN-N20, symbol Power_Management:TPS22993
Connections:
- new net +3V3: C19.1, C20.1, U7.10 (ON1), U7.12 (VIN4), U7.14 (VIN3), U7.18 (VDD), U7.2 (VIN2), U7.4 (VIN1), U7.6 (ADD1), U7.7 (ON4), U7.8 (ON3), U7.9 (ON2), U8.10 (ON1), U8.12 (VIN4), U8.14 (VIN3), U8.18 (VDD), U8.2 (VIN2), U8.4 (VIN1), U8.7 (ON4), U8.8 (ON3), U8.9 (ON2)
- new net FACE0_POWER: U7.5 (VOUT1)
- new net FACE1_POWER: U7.1 (VOUT2)
- new net FACE2_POWER: U7.15 (VOUT3)
- new net FACE3_POWER: U7.11 (VOUT4)
- new net FACE4_POWER: U8.5 (VOUT1)
- new net GND: C19.2, C20.2, U7.13 (GND), U7.16 (ADD2), U7.20 (ADD3), U8.13 (GND), U8.16 (ADD2), U8.20 (ADD3), U8.6 (ADD1)
- new net SCL1: U7.17 (SCL), U8.17 (SCL)
- new net SDA1: U7.19 (SDA), U8.19 (SDA)
- new net VBUSP: U7.3 (VBIAS), U8.3 (VBIAS)
Other:
- note added: "I2C Load Switch Read Address: 0xE0 Write Address: 0xE1"
- note added: "I2C Load Switch Read Address: 0xE2 Write Address: 0xE3"
