File: FC_V6/power_block_diagram.kicad_sch (KiCad schematic)
At the start: 0 parts

Commit message: V6: Checkpoint
Changed lines of the file:
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@@
 	(paper "A4")
 	(rectangle
-		(start 49.53 100.838)
-		(end 67.31 111.76)
-		(stroke
-			(width 0)
-			(type solid)
-		)
-		(fill
-			(type color)
-			(color 145 255 190 1)
-		)
-	)
-	(rectangle
-		(start 49.53 79.248)
-		(end 67.31 90.17)
+		(start 50.8 100.838)
+		(end 68.58 111.76)
+		(stroke
+			(width 0)
+			(type solid)
+		)
+		(fill
+			(type color)
+			(color 145 255 190 1)
+		)
+	)
+	(rectangle
+		(start 50.8 79.248)
+		(end 68.58 90.17)
 		(stroke
 			(width 0)
@@
 	)
 	(rectangle
-		(start 49.53 132.588)
-		(end 67.31 143.51)
+		(start 50.8 132.588)
+		(end 68.58 143.51)
 		(stroke
 			(width 0)
@@
 	(text "Power Monitor 4\n"
 		(exclude_from_sim no)
-		(at 58.42 106.68 0)
+		(at 59.69 106.68 0)
 		(effects
 			(font
@@
 	(text "Power Monitor 5"
 		(exclude_from_sim no)
-		(at 58.42 138.43 0)
+		(at 59.69 138.43 0)
 		(effects
 			(font
@@
 	(text "Power Monitor 3"
 		(exclude_from_sim no)
-		(at 58.42 85.09 0)
+		(at 59.69 85.09 0)
 		(effects
 			(font
@@
 	(polyline
 		(pts
+			(xy 43.18 138.43) (xy 50.8 138.43)
+		)
+		(stroke
+			(width 0)
+			(type default)
+		)
+	)
+	(polyline
+		(pts
 			(xy 68.58 53.34) (xy 81.28 53.34)
 		)
@@
 	(polyline
 		(pts
+			(xy 43.18 85.09) (xy 50.8 85.09)
+		)
+		(stroke
+			(width 0)
+			(type default)
+		)
+	)
+	(polyline
+		(pts
 			(xy 68.58 31.496) (xy 81.28 31.496)
 		)
@@
 		)
 		(stroke
+			(width 0)
+			(type default)
+		)
+	)
+	(polyline
+		(pts
+			(xy 43.18 106.68) (xy 50.8 106.68)
+		)
+		(stroke
