File: FC_V6/stm32_mcu.kicad_sch (KiCad schematic)
At the start: 0 parts

Commit message: V6: Checkpoint
Parts:
- added U1: STM32U5A5QJIxQ, Package_BGA:UFBGA-132_7x7mm_Layout12x12_P0.5mm, symbol MCU_ST_STM32U5:STM32U5A5QJIxQ
Connections:
- new net: U1.E4 (VSS), U1.E9 (VSS), U1.F6 (VSS), U1.G7 (VSS), U1.H4 (VSS), U1.H9 (VSS)
