File: FC_V6/USB_HUB.kicad_sch (KiCad schematic)
At the start: 20 parts, among them J1 USB_C_Receptacle_USB2.0_16P, U4 TPD4EUSB30, U5 CH334F, Y1 12Mhz

Commit message: Finished MPPT Power Train with place holder buck converters, fixed minor error with OCTOSPI power supply
Parts:
- removed D1: 1N5819HW-7-F, Diode_SMD:D_SOD-123, symbol Device:D
- added C64: 12pF, Capacitor_SMD:C_0402_1005Metric, symbol Device:C_Small_US
- added D11, D12, D2: SS14, Diode_SMD:D_SMA, symbol Diode:SS14
- added R28: 200K, Resistor_SMD:R_0402_1005Metric, symbol Device:R_Small_US
- added R29: 1k, Resistor_SMD:R_0402_1005Metric, symbol Device:R_Small_US
- added U13: CH221K, CH221K:SOT95P280X120-6N, symbol CH221K:CH221K
- renumbered C19 to C20, C20 to C21, C21 to C22, C22 to C23, C23 to C24, D2 to D3, D3 to D4, D4 to D5, D5 to D6, D6 to D7
Connections:
- net GND: now also C64.2, U13.2 (GND)
- net at J1.A5 (CC1), R2.1: now also U13.4 (CC1)
- net at J1.A4 (VBUS), J1.A9 (VBUS), J1.B4 (VBUS)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: now also D11.2 (A), D12.2 (A), D2.2 (A), R29.2
- net at J1.B5 (CC2), R3.1: now also U13.5 (CC2)
- new net: R28.1, U13.6 (CFG)
- new net: C64.1, R28.2, R29.1, U13.1 (VDD)
- new net +VBUS: D11.1 (K), D12.1 (K), D2.1 (K)
- no-connect marks 9 -> 10
Other:
- note added: "+20V VBUS!"
- title: (none) -> USB Hub + PD
