File: FC_V5e_Production_Rev2/FC_V5e_Production_Rev2.kicad_sch (KiCad schematic)
At the start: 72 parts, among them IC3 RV-3028-C7_32.768kHz_1ppm_TA_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, J12 USB_C_Receptacle_USB2.0_16P, J16 DEBUG, J18 Payload, J22 SWD Port, J3 Life Makes Lemonade, J5 BM04B-SRSS-TB(LF)(SN), SW1 KMR2, SW2 KMR2, U13 E22-400M30S, U15 LIS2MDL, U2 ZDSD04GLGEAG, U3 TCA9548APWR, U30 E28-2G4M27S, U7 LSM6DSOTR

Commit message: V5e_Rev2: Design review fixes and JLCPCB BOM corrections
Layout
- Move C10 (PSRAM bypass) back to (210.5, 74), the V5d flight position.
  Commit 066aeb7 had nudged it 0.125 mm to clear the new U5 courtyard,
  leaving its stubs behind and creating 4 clearance errors (worst
  0.089 mm +3V3 to GND). Trim U5 B.CrtYd start-x -2.82 -> -2.65 instead.
  DRC back to Rev1 baseline: 35 clearance (all inherited pad-pitch), 1
  courtyard (SW2/TP2), none near C10/U5.

Schematic
- Remove orphan ~{5V_RESET} global label on U9 GPB6, place no-connect.
- U10 value/MPN TPS54226PWPR -> TPS54225PWPR to match the part built and
  validated on Rev1 (C555460). Same fsw, D-CAP2, pinout, Table 1 values;
  54226 only adds light-load skip and has been out of stock since Feb.
- U2 ZDSD04GLGEAG -> ZDSD02GLGEAG (C2875853). 4 Gb SKU is out of stock;
  2 Gb is same family, datasheet, land pattern. Firmware has no capacity
  dependence. Revisit 4 Gb (MKDV4GIL-AST) in a future rev.
- IC3 value/MPN RV-3028-C7 QC -> QA to match the assigned C3304278.
  QA/QC is qualification grade (AEC-Q200 vs commercial), same die and
  same 1 ppm spec. Mouser fields still point at the QC part, which
  remains an acceptable alternate.

jlcpcb/project.db (plugin BOM/CPL source)
- Add U5 -> C18214056, C10 -> C1525, R37 -> C25744 (all Rev2-new, were
  missing and would have been left unplaced).
- J7/J10/J19/J20 C2692098 (stock 0) -> C506665 DF11-4DP-2DSA(08), the
  same vertical receptacle with a different plating suffix.
- U1 C33503485 (TLV1824DR, SOIC-14, wrong device and package) ->
  C181596 TLV1704AIPWR TSSOP-14. Rev1 as-ordered carried the wrong part.
- D7 C2128 (1N4148WS) -> C17429783 (1N4151WS-E3-18) so the build matches
  the schematic and the "D7 MUST be 1N4151WS" watchdog note.
- U2 -> C2875853, IC3 value synced.

ERC violation set unchanged apart from the removed orphan label.

Co-Authored-By: Claude Fable 5.1 <noreply@anthropic.com>
Claude-Session: https://claude.ai/code/session_01ALRFkyTuqxnA412gooXH2e
Parts:
- IC3: value RV-3028-C7_32.768kHz_1ppm_TA_QC -> RV-3028-C7_32.768kHz_1ppm_TA_QA; Manufacturer_Part_Number RV-3028-C7 32.768kHz 1ppm TA QC -> RV-3028-C7 32.768kHz 1ppm TA QA
- U2: value ZDSD04GLGEAG -> ZDSD02GLGEAG; LCSC Part C2875854 -> C2875853
Changed lines of the file:
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@@
 			)
 		)
-		(property "Value" "RV-3028-C7_32.768kHz_1ppm_TA_QC"
+		(property "Value" "RV-3028-C7_32.768kHz_1ppm_TA_QA"
 			(at 128.016 222.25 0)
 			(show_name no)
@@
 			)
 		)
-		(property "Manufacturer_Part_Number" "RV-3028-C7 32.768kHz 1ppm TA QC"
+		(property "Manufacturer_Part_Number" "RV-3028-C7 32.768kHz 1ppm TA QA"
 			(at 143.51 1022.25 0)
 			(hide yes)
@@
 			)
 		)
-		(property "Value" "ZDSD04GLGEAG"
+		(property "Value" "ZDSD02GLGEAG"
 			(at 49.53 231.14 0)
 			(show_name no)
@@
 			)
 		)
-		(property "LCSC Part" "C2875854"
+		(property "LCSC Part" "C2875853"
 			(at 50.8 254 0)
 			(hide yes)

Commit message: V5e_Rev2: Normalize value strings and add connector MPN fields
JLCPCB Tools flagged identical LCSC numbers carrying different value
strings. Normalize to one convention across all sheets:
- Resistors: lowercase k (100K -> 100k, 10K, 4.7K, 22.1K, 243K, 73.2K)
- Capacitors: <value><prefix>F (100n/100nf -> 100nF, 220nF, 10nF, 10pF,
  15pF, 10uF, 4.7uF)
- D13 DFLS130L-7 -> DFLS130L to match D12/D15
- Hidden MPN property on the 23 connectors with an LCSC assignment

Board updated from schematic so footprint values match. project.db
values synced and LCSC assignments restored after the plugin cleared
rows whose value changed. ERC violation set unchanged.

Co-Authored-By: Claude Fable 5.1 <noreply@anthropic.com>
Claude-Session: https://claude.ai/code/session_01ALRFkyTuqxnA412gooXH2e
Parts:
- C18, C26, C28, C32, C34, C35: value 100nf -> 100nF
- C31: value 220nf -> 220nF
- J12: MPN (none) -> TYPE-C-31-M-12
- J16, J18: MPN (none) -> DF11-12DP-2DSA(08)
- J22: MPN (none) -> BM03B-SRSS-TB(LF)(SN)
- J5: MPN (none) -> BM04B-SRSS-TB(LF)(SN)
- R15: value 10K -> 10k
Changed lines of the file:
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@@
 			)
 		)
-		(property "Value" "220nf"
+		(property "Value" "220nF"
 			(at 368.06 58.44 90)
 			(show_name no)
@@
 			)
 		)
-		(property "Value" "100nf"
+		(property "Value" "100nF"
 			(at 293.13 58.44 90)
 			(show_name no)
@@
 			)
 		)
-		(property "Value" "100nf"
+		(property "Value" "100nF"
 			(at 230.519 49.804 90)
 			(show_name no)
@@
 			)
 		)
-		(property "Value" "100nf"
+		(property "Value" "100nF"
 			(at 73.42 229.89 90)
 			(show_name no)
@@
 			)
 		)
+		(property "MPN" "DF11-12DP-2DSA(08)"
+			(at 113.03 269.24 0)
+			(hide yes)
+			(show_name no)
+			(do_not_autoplace no)
+			(effects
+				(font
+					(size 1.27 1.27)
+				)
+			)
+		)
 		(property "Datasheet" ""
 			(at 113.03 269.24 0)
@@
 			)
 		)
-		(property "Value" "100nf"
+		(property "Value" "100nF"
 			(at 161.05 237.51 90)
 			(show_name no)
@@
 			)
 		)
-		(property "Value" "100nf"
+		(property "Value" "100nF"
 			(at 368.06 34.31 90)
 			(show_name no)
@@
 			)
 		)
-		(property "Value" "10K"
+		(property "Value" "10k"
 			(at 301.244 92.075 90)
 			(show_name no)
@@
 			)
 		)
+		(property "MPN" "BM04B-SRSS-TB(LF)(SN)"
+			(at 46.99 270.51 0)
+			(hide yes)
+			(show_name no)
+			(do_not_autoplace no)
+			(effects
+				(font
+					(size 1.27 1.27)
+				)
+			)
+		)
 		(property "Datasheet" ""
 			(at 46.99 270.51 0)
@@
 			)
 		)
+		(property "MPN" "TYPE-C-31-M-12"
+			(at 161.29 38.1 0)
+			(hide yes)
+			(show_name no)
+			(do_not_autoplace no)
+			(effects
+				(font
+					(size 1.27 1.27)
+				)
+			)
+		)
 		(property "Datasheet" "https://www.usb.org/sites/default/files/documents/usb_type-c.zip"
 			(at 161.29 38.1 0)
@@
 			)
 		)
+		(property "MPN" "DF11-12DP-2DSA(08)"
+			(at 158.75 267.97 0)
+			(hide yes)
+			(show_name no)
+			(do_not_autoplace no)
+			(effects
+				(font
+					(size 1.27 1.27)
+				)
+			)
+		)
 		(property "Datasheet" ""
 			(at 158.75 267.97 0)
@@
 			)
 		)
+		(property "MPN" "BM03B-SRSS-TB(LF)(SN)"
+			(at 114.3 36.83 0)
+			(hide yes)
+			(show_name no)
+			(do_not_autoplace no)
+			(effects
+				(font
+					(size 1.27 1.27)
+				)
+			)
+		)
 		(property "Datasheet" ""
 			(at 114.3 36.83 0)
@@
 			)
 		)
-		(property "Value" "100nf"
+		(property "Value" "100nF"
 			(at 173.75 237.51 90)
 			(show_name no)
