File: FC_V5e_Production_Rev2/load_switches.kicad_sch (KiCad schematic)
At the start: 53 parts, among them U19 AP22653AW6-7, U21 AP22653AW6-7, U22 AP22653AW6-7, U23 AP22653AW6-7, U24 AP22653AW6-7, U25 TPS2HB50AQPWPRQ1, U27 AP22653AW6-7, U29 AP22653AW6-7, U6 TPS4H160AQPWPRQ1

Commit message: V5e_Rev2: Normalize value strings and add connector MPN fields
JLCPCB Tools flagged identical LCSC numbers carrying different value
strings. Normalize to one convention across all sheets:
- Resistors: lowercase k (100K -> 100k, 10K, 4.7K, 22.1K, 243K, 73.2K)
- Capacitors: <value><prefix>F (100n/100nf -> 100nF, 220nF, 10nF, 10pF,
  15pF, 10uF, 4.7uF)
- D13 DFLS130L-7 -> DFLS130L to match D12/D15
- Hidden MPN property on the 23 connectors with an LCSC assignment

Board updated from schematic so footprint values match. project.db
values synced and LCSC assignments restored after the plugin cleared
rows whose value changed. ERC violation set unchanged.

Co-Authored-By: Claude Fable 5.1 <noreply@anthropic.com>
Claude-Session: https://claude.ai/code/session_01ALRFkyTuqxnA412gooXH2e
Parts:
- C38, C44, C47, C48, C49, C50, C51, C52, C53, C55, C59, C60, C79, C80: value 100nf -> 100nF
- C54, C56, C57, C58: value 220nf -> 220nF
- R100, R103, R104: value 4.7K -> 4.7k
Changed lines of the file:
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@@
 			)
 		)
-		(property "Value" "4.7K"
+		(property "Value" "4.7k"
 			(at 213.614 84.836 0)
 			(show_name no)
@@
 			)
 		)
-		(property "Value" "100nf"
+		(property "Value" "100nF"
 			(at 81.04 115.59 90)
 			(show_name no)
@@
 			)
 		)
-		(property "Value" "220nf"
+		(property "Value" "220nF"
 			(at 275.59 116.586 90)
 			(show_name no)
@@
 			)
 		)
-		(property "Value" "220nf"
+		(property "Value" "220nF"
 			(at 260.35 116.586 90)
 			(show_name no)
@@
 			)
 		)
-		(property "Value" "220nf"
+		(property "Value" "220nF"
 			(at 265.43 116.586 90)
 			(show_name no)
@@
 			)
 		)
-		(property "Value" "100nf"
+		(property "Value" "100nF"
 			(at 49.29 69.87 90)
 			(show_name no)
@@
 			)
 		)
-		(property "Value" "4.7K"
+		(property "Value" "4.7k"
 			(at 213.614 79.756 0)
 			(show_name no)
@@
 			)
 		)
-		(property "Value" "220nf"
+		(property "Value" "220nF"
 			(at 270.51 116.586 90)
 			(show_name no)
@@
 			)
 		)
-		(property "Value" "100nf"
+		(property "Value" "100nF"
 			(at 49.29 43.2 90)
 			(show_name no)
@@
 			)
 		)
-		(property "Value" "100nf"
+		(property "Value" "100nF"
 			(at 81.04 142.26 90)
 			(show_name no)
@@
 			)
 		)
-		(property "Value" "100nf"
+		(property "Value" "100nF"
 			(at 242.33 147.34 90)
 			(show_name no)
@@
 			)
 		)
-		(property "Value" "100nf"
+		(property "Value" "100nF"
 			(at 49.29 95.27 90)
 			(show_name no)
@@
 			)
 		)
-		(property "Value" "100nf"
+		(property "Value" "100nF"
 			(at 49.29 123.21 90)
 			(show_name no)
@@
 			)
 		)
-		(property "Value" "100nf"
+		(property "Value" "100nF"
 			(at 81.04 35.58 90)
 			(show_name no)
@@
 			)
 		)
-		(property "Value" "100nf"
+		(property "Value" "100nF"
 			(at 210.58 154.96 90)
 			(show_name no)
@@
 			)
 		)
-		(property "Value" "100nf"
+		(property "Value" "100nF"
 			(at 81.04 62.25 90)
 			(show_name no)
@@
 			)
 		)
-		(property "Value" "100nf"
+		(property "Value" "100nF"
 			(at 49.29 149.88 90)
 			(show_name no)
@@
 			)
 		)
-		(property "Value" "100nf"
+		(property "Value" "100nF"
 			(at 81.04 87.65 90)
 			(show_name no)
@@
 			)
 		)
-		(property "Value" "100nf"
+		(property "Value" "100nF"
 			(at 81.04 174.01 90)
 			(show_name no)
@@
 			)
 		)
-		(property "Value" "100nf"
+		(property "Value" "100nF"
 			(at 49.29 181.63 90)
 			(show_name no)
@@
 			)
 		)
-		(property "Value" "4.7K"
+		(property "Value" "4.7k"
 			(at 214.122 92.71 0)
 			(show_name no)
