File: FlatSat_V1/solar_power_injection.kicad_sch (KiCad schematic)
At the start: 11 parts, among them J400 Terminal_2P_5.08mm, J401 Terminal_2P_5.08mm

Commit message: FlatSat V1: apply pre-order review fix-this-rev items 1,2,3,4,6,7
1 Mode 2 feeds the FC from BQ25886 SYS (JP510.1 -> CHG_SYS), 78 -> 24 mOhm.
2 Dir_Chrg_In attaches at J14.1 (In1 1.5 mm L11 stub); J16.8 stub and
  its 140 mm / 5-via run removed. J500.1->J14.1 307 -> 35 mOhm.
3 Replica sense-loop copper 68 -> 8 mOhm; excess-discharge trip
  ~2.3 A -> ~7.7 A. Kelvin VSS tap at Q500 source.
4 BQ25886: C513 at the SYS pins, 9 EP thermal PTH pads (U18 convention),
  GND vias at every charger cap, SW 0.8 mm, PMID 1.0 mm on F.Cu.
6 bench_power_width DRC rule (warning, outside FC_COPY), 7 power nodes
  labelled into BenchPower, BenchPower5V for CHG_DVIN.
7 VSOLAR bench hard maximum 18 V (heritage C40 is 10 V), 18V MAX silk.

Gates: heritage refill 0, attachment 0/7/37, DRC 14/1/11, ERC 12,
via-in-pad 7. Edit scripts kept under review_fixes_scripts/.

Co-Authored-By: Claude Opus 5.5 (1M context) <noreply@anthropic.com>
Connections:
- net INJ_A_PTC: now reaches D400.2 (A), F400.2
- net INJ_B_OR: now reaches D401.1 (K), JP401.1 (A)
- net INJ_B_PTC: now reaches D401.2 (A), F401.2
- net INJ_A_OR: now reaches D400.1 (K), JP400.1 (A)
Other:
- note added: "Bench PSU setting: 12 V to 18 V nominal, HARD MAXIMUM 18 V (heritage C40, the LT3652 VIN bypass on V_SOLAR_SENSE, is a 10 V X5R). INA219 U8 (0x41) IN+"
- note added: "HARD MAXIMUM 18 V procedure: set PSU OVP <= 18 V and verify the trip with J400/J401 disconnected (raise the output until OVP trips) before each session; do not soak at 18 V."
- note added: "IC6 R75 = 0.1 ohm sets the LT3652 1.0 A charge current) -- 28 % margin. 33 V Vmax leaves 15 V over the 18 V hard maximum. Itrip (3.70 A)"
- note added: "Secondary limits only: INA219 U8 26 V absolute maximum, F400/F401 33 V Vmax. The 18 V ceiling exists because a shorted 10 V C40 would dump PSU/PTC current into FC-copy copper."
- note removed: "Bench PSU setting: 12 V to 18 V nominal, HARD MAXIMUM 24 V (brief section 6.3; F400/F401 are 33 V Vmax, so 9 V of margin). INA219 U8 (0x41) IN+"
- note removed: "IC6 R75 = 0.1 ohm sets the LT3652 1.0 A charge current) -- 28 % margin. 33 V Vmax leaves 9 V over the brief's 24 V hard maximum. Itrip (3.70 A)"
Changed lines of the file:
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@@
 		)
 	)
-	(text "Bench PSU setting: 12 V to 18 V nominal, HARD MAXIMUM 24 V (brief section 6.3; F400/F401 are 33 V Vmax, so 9 V of margin). INA219 U8 (0x41) IN+"
+	(text "Bench PSU setting: 12 V to 18 V nominal, HARD MAXIMUM 18 V (heritage C40, the LT3652 VIN bypass on V_SOLAR_SENSE, is a 10 V X5R). INA219 U8 (0x41) IN+"
 		(exclude_from_sim no)
 		(at 20 160 0)
@@
 		)
 	)
-	(text "IC6 R75 = 0.1 ohm sets the LT3652 1.0 A charge current) -- 28 % margin. 33 V Vmax leaves 9 V over the brief's 24 V hard maximum. Itrip (3.70 A)"
+	(text "IC6 R75 = 0.1 ohm sets the LT3652 1.0 A charge current) -- 28 % margin. 33 V Vmax leaves 15 V over the 18 V hard maximum. Itrip (3.70 A)"
 		(exclude_from_sim no)
 		(at 20 208.67 0)
@@
 		(effects
 			(font
+				(size 1.27 1.27)
+			)
+			(justify left bottom)
+		)
+	)
+	(text "HARD MAXIMUM 18 V procedure: set PSU OVP <= 18 V and verify the trip with J400/J401 disconnected (raise the output until OVP trips) before each session; do not soak at 18 V."
+		(exclude_from_sim no)
+		(at 20 251.34 0)
+		(effects
+			(font
+				(size 1.27 1.27)
+			)
+			(justify left bottom)
+		)
+	)
+	(text "Secondary limits only: INA219 U8 26 V absolute maximum, F400/F401 33 V Vmax. The 18 V ceiling exists because a shorted 10 V C40 would dump PSU/PTC current into FC-copy copper."
+		(exclude_from_sim no)
+		(at 20 253.34 0)
+		(effects
+			(font
+				(size 1.27 1.27)
+			)
+			(justify left bottom)
+		)
+	)
+	(label "INJ_A_PTC"
+		(at 130.81 76.2 0)
+		(effects
+			(font
+				(size 1.27 1.27)
+			)
+			(justify left bottom)
+		)
+	)
+	(label "INJ_A_OR"
+		(at 168.91 76.2 0)
+		(effects
+			(font
+				(size 1.27 1.27)
+			)
+			(justify left bottom)
+		)
+	)
+	(label "INJ_B_PTC"
+		(at 130.81 139.7 0)
+		(effects
+			(font
+				(size 1.27 1.27)
+			)
+			(justify left bottom)
+		)
+	)
+	(label "INJ_B_OR"
+		(at 168.91 139.7 0)
+		(effects
+			(font
