File: FC_V5e_Production_Rev3/eps_side.kicad_sch (KiCad schematic)
At the start: 69 parts, among them IC6 LT3652IMSE#PBF, J1 Conn_01x06, J10 INHIBIT_P2, J11 Conn_01x06, J13 Conn_01x06, J14 Battery Input, J15 ISS_INHIBIT_Picolock, J19 ISS_INHIBIT, J2 Conn_01x06, J20 RBF_Inhibit, J21 Heater Output, J23 Aux Deploy 1, J24 Deploy 2, J29 INHIBIT_S2_Picolock, J30 RBF_Picolock, J6 Conn_01x06, J7 INHIBIT_P1, J8 INHIBIT_S1_Picolock, J9 Conn_01x06, U10 TPS54225PWPR, U12 LT8610ABEMSE#TRPBF, U16 INA219AxDCN, U8 INA219AxDCN, U9 MCP23017_SS

Commit message: V5e_Rev3: Tie U12 LT8610AB SYNC to GND (Burst Mode)
SYNC was left floating. Grounding it selects Burst Mode, the
datasheet's low-quiescent-current light-load mode and the ADI demo
board default, instead of leaving the mode to an undefined input.
Schematic: GND symbol on pin 1. PCB: 0.2 mm B.Cu stub from pad 1 into
the exposed GND pad; zones refilled. Only U12 pin 1 changes net.

Co-Authored-By: Claude Opus 5.5 (1M context) <noreply@anthropic.com>
Connections:
- net GND: now also U12.1 (SYNC)
Changed lines of the file:
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@@
+		)
+	)
+	(wire
+		(pts
+			(xy 318.77 138.43) (xy 313.69 138.43)
+		)
+		(stroke
+			(width 0)
+			(type default)
 		)
 	)
 	(symbol
+		(lib_id "power:GND")
+		(at 313.69 138.43 270)
+		(unit 1)
+		(body_style 1)
+		(exclude_from_sim no)
+		(in_bom yes)
+		(on_board yes)
+		(in_pos_files yes)
+		(dnp no)
+		(fields_autoplaced yes)
+		(property "Reference" "#PWR0173"
+			(at 307.34 138.43 0)
+			(hide yes)
+			(show_name no)
+			(do_not_autoplace no)
+			(effects
+				(font
+					(size 1.27 1.27)
+				)
+			)
+		)
+		(property "Value" "GND"
+			(at 309.88 138.43 0)
+			(show_name no)
+			(do_not_autoplace no)
+			(effects
+				(font
+					(size 1.27 1.27)
+				)
+			)
+		)
+		(property "Footprint" ""
+			(at 313.69 138.43 0)
+			(hide yes)
+			(show_name no)
+			(do_not_autoplace no)
+			(effects
+				(font
+					(size 1.27 1.27)
+				)
+			)
+		)
+		(property "Datasheet" ""
+			(at 313.69 138.43 0)
+			(hide yes)
+			(show_name no)
+			(do_not_autoplace no)
+			(effects
+				(font
+					(size 1.27 1.27)
+				)
+			)
+		)
+		(property "Description" ""
+			(at 313.69 138.43 0)
+			(hide yes)
+			(show_name no)
+			(do_not_autoplace no)
+			(effects
+				(font
+					(size 1.27 1.27)
+				)
+			)
+		)
+		(pin "1"
+		)
+		(instances
+			(project "FC_V5e_Production_Rev3"
+				(path "/c64c0d72-a9f6-4f3a-891e-1f647558f538/7cbc73fc-c188-4597-842f-d15f69db7471"
+					(reference "#PWR0173")
+					(unit 1)
+				)
+			)
+		)
+	)	(symbol
 		(lib_id "Adafruit ItsyBitsy RP2040-eagle-import:CAP_CERAMIC_0402NO")
 		(at 356.87 149.86 270)
