File: FC_V5e_Production_Rev3/watchdog.kicad_sch (KiCad schematic)
At the start: 31 parts, among them J4 Conn_01x02, U1 TLV1704

Commit message: V5e_Rev3: Remove watchdog enable jumper JP6
JP6 was an open solder jumper between the watchdog comparator output
(U1 pin 13) and the 3V3 regulator reset (~3v3_RESET). It let CircuitPython
boards flash firmware that could not pet the watchdog inside its window.
F Prime starts petting the watchdog early enough, and an unbridged JP6 on
a flight unit silently disables the power-cycle path.

Schematic: JP6 replaced with a wire. PCB: JP6 footprint removed, a 0.3 mm
F.Cu trace joins the two existing stubs, and U1 pin 13 moves onto
~3v3_RESET. project.db: JP6 row dropped. DRC and schematic parity counts
match Rev2 exactly (50 items, all pre-existing).

Co-Authored-By: Claude Opus 5.5 (1M context) <noreply@anthropic.com>
Parts:
- removed JP6: SolderJumper_2_Open, Jumper:SolderJumper-2_P1.3mm_Open_RoundedPad1.0x1.5mm, symbol Jumper:SolderJumper_2_Open
Connections:
- net ~{3v3_RESET}: now also U1.13
Changed lines of the file:
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@@
 		)
 	)
-	(symbol
-		(lib_id "Jumper:SolderJumper_2_Open")
-		(at 269.24 128.27 270)
-		(unit 1)
-		(body_style 1)
-		(exclude_from_sim no)
-		(in_bom yes)
-		(on_board yes)
-		(in_pos_files yes)
-		(dnp no)
-		(property "Reference" "JP6"
-			(at 266.446 128.524 0)
-			(show_name no)
-			(do_not_autoplace no)
-			(effects
-				(font
-					(size 1.27 1.27)
-				)
-			)
+	(wire
+		(pts
+			(xy 269.24 124.46) (xy 269.24 132.08)
 		)
-		(property "Value" "SolderJumper_2_Open"
-			(at 283.21 128.27 90)
-			(hide yes)
-			(show_name no)
-			(do_not_autoplace no)
-			(effects
-				(font
-					(size 1.27 1.27)
-				)
-			)
-		)
-		(property "Footprint" "Jumper:SolderJumper-2_P1.3mm_Open_RoundedPad1.0x1.5mm"
-			(at 269.24 128.27 0)
-			(hide yes)
-			(show_name no)
-			(do_not_autoplace no)
-			(effects
-				(font
-					(size 1.27 1.27)
-				)
-			)
-		)
-		(property "Datasheet" ""
-			(at 269.24 128.27 0)
-			(hide yes)
-			(show_name no)
-			(do_not_autoplace no)
-			(effects
-				(font
-					(size 1.27 1.27)
-				)
-			)
-		)
-		(property "Description" ""
-			(at 269.24 128.27 0)
-			(hide yes)
-			(show_name no)
-			(do_not_autoplace no)
-			(effects
-				(font
-					(size 1.27 1.27)
-				)
-			)
-		)
-		(pin "1"
-		)
-		(pin "2"
-		)
-		(instances
-			(project "FC_V5e_Production_Rev3"
-				(path "/c64c0d72-a9f6-4f3a-891e-1f647558f538/d3e26510-981a-4dd5-9b7d-a587e6324dc6"
-					(reference "JP6")
-					(unit 1)
-				)
-			)
+		(stroke
+			(width 0)
+			(type default)
 		)
 	)

Commit message: V5e_Rev3: Drop stale 'WDT enabled when soldered' note
The note labelled JP6, which the previous commit removed.

Co-Authored-By: Claude Opus 5.5 (1M context) <noreply@anthropic.com>
Other:
- note removed: "WDT enabled when soldered"
Changed lines of the file:
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@@
-		)
-	)
-	(text "WDT enabled\nwhen soldered"
-		(exclude_from_sim no)
-		(at 271.399 130.048 0)
-		(effects
-			(font
-				(size 0.889 0.889)
-			)
-			(justify left bottom)
 		)
 	)

Commit message: V5e_Rev3: Watchdog timing caps C21-C23 to 25 V X5R (C96446)
The watchdog sheet note requires 15-25 V on C21, C22 and C23, but
project.db assigned C19702, a 10 V part. C96446 (Samsung
CL10A106MA8NRNC, 10 uF 25 V X5R 0603) is a Basic part on the same
footprint. Schematic MPN/MFR/description fields updated to match.

Co-Authored-By: Claude Opus 5.5 (1M context) <noreply@anthropic.com>
Parts:
- C21, C22, C23: DPN 490-12317-1-ND -> C96446; DST Digi-Key -> LCSC; MFR Murata -> Samsung Electro-Mechanics; MPN GRT188R61C106KE13D -> CL10A106MA8NRNC
Changed lines of the file:
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@@
 			)
 		)
-		(property "Description" "10 µF ±10% 16V Ceramic Capacitor X5R 0603 (1608 Metric)"
+		(property "Description" "10 µF ±20% 25V Ceramic Capacitor X5R 0603 (1608 Metric)"
 			(at 180.34 128.27 0)
 			(hide yes)
@@
 			)
 		)
-		(property "DPN" "490-12317-1-ND"
+		(property "DPN" "C96446"
 			(at 180.34 128.27 0)
 			(hide yes)
@@
 			)
 		)
-		(property "DST" "Digi-Key"
+		(property "DST" "LCSC"
 			(at 180.34 128.27 0)
 			(hide yes)
@@
 			)
 		)
-		(property "MFR" "Murata"
+		(property "MFR" "Samsung Electro-Mechanics"
 			(at 180.34 128.27 0)
 			(hide yes)
@@
 			)
 		)
-		(property "MPN" "GRT188R61C106KE13D"
+		(property "MPN" "CL10A106MA8NRNC"
 			(at 180.34 128.27 0)
 			(hide yes)
@@
 			)
 		)
-		(property "Description" "10 µF ±10% 16V Ceramic Capacitor X5R 0603 (1608 Metric)"
+		(property "Description" "10 µF ±20% 25V Ceramic Capacitor X5R 0603 (1608 Metric)"
 			(at 170.18 128.27 0)
 			(hide yes)
@@
 			)
 		)
-		(property "DPN" "490-12317-1-ND"
+		(property "DPN" "C96446"
 			(at 170.18 128.27 0)
 			(hide yes)
@@
 			)
 		)
-		(property "DST" "Digi-Key"
+		(property "DST" "LCSC"
 			(at 170.18 128.27 0)
 			(hide yes)
@@
 			)
 		)
-		(property "MFR" "Murata"
+		(property "MFR" "Samsung Electro-Mechanics"
 			(at 170.18 128.27 0)
 			(hide yes)
@@
 			)
 		)
-		(property "MPN" "GRT188R61C106KE13D"
+		(property "MPN" "CL10A106MA8NRNC"
 			(at 170.18 128.27 0)
 			(hide yes)
@@
 			)
 		)
-		(property "Description" "10 µF ±10% 16V Ceramic Capacitor X5R 0603 (1608 Metric)"
+		(property "Description" "10 µF ±20% 25V Ceramic Capacitor X5R 0603 (1608 Metric)"
 			(at 135.89 125.73 0)
 			(hide yes)
@@
 			)
 		)
-		(property "DPN" "490-12317-1-ND"
+		(property "DPN" "C96446"
 			(at 135.89 125.73 0)
 			(hide yes)
@@
 			)
 		)
-		(property "DST" "Digi-Key"
+		(property "DST" "LCSC"
 			(at 135.89 125.73 0)
 			(hide yes)
@@
 			)
 		)
-		(property "MFR" "Murata"
+		(property "MFR" "Samsung Electro-Mechanics"
 			(at 135.89 125.73 0)
 			(hide yes)
@@
 			)
 		)
-		(property "MPN" "GRT188R61C106KE13D"
+		(property "MPN" "CL10A106MA8NRNC"
 			(at 135.89 125.73 0)
 			(hide yes)

Commit message: V5e_Rev3: Remove unplaced watchdog test points TP9-TP13
TP9-TP13 were on the watchdog sheet but never placed on the PCB, so
they only produced missing_footprint parity errors. The circuit is
trusted from Rev1/Rev2 test, so the test points are dropped rather than
placed. Nets are unchanged (the test points sat in-line on existing
wire junctions). ERC 460 -> 450; DRC parity loses the 5 missing items.

Co-Authored-By: Claude Opus 5.5 (1M context) <noreply@anthropic.com>
Parts:
- removed TP10, TP11, TP12, TP13, TP9: TestPoint-MinTH, oresat-misc:TestPoint-0.75mm-th, symbol oresat-misc:Test-Point-0.75mm-th
